File: 0002-clap-detector/0002-clap-detector.kicad_pcb (KiCad board)
At the start: 2 copper layers, 58 x 37 mm, 49 parts, among them J1 9V, J2 OUT, K1 HF49FD 012-1H11, Q1 BC847B, Q2 BC847B, Q3 BCV26, Q4 BC847B, U1 4017

Commit message: Small corrections
Routing:
- net Net-(D3-A): track 18.1 -> 27.5 mm
Changed lines of the file:
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@@
 	)
 	(segment
-		(start 129.9 93.9)
+		(start 129.9 110.7)
+		(end 128.8 109.6)
+		(width 0.4)
+		(layer "B.Cu")
+		(net 1)
+	)
+	(segment
+		(start 128.8 109.6)
+		(end 128.8 92.8)
+		(width 0.4)
+		(layer "B.Cu")
+		(net 1)
+	)
+	(segment
+		(start 128.8 92.8)
 		(end 126 90)
-		(width 0.4)
-		(layer "B.Cu")
-		(net 1)
-	)
-	(segment
-		(start 129.9 110.7)
-		(end 129.9 93.9)
 		(width 0.4)
 		(layer "B.Cu")
@@
 	)
 	(segment
+		(start 166.4925 89.9925)
+		(end 170.2 93.7)
+		(width 1)
+		(layer "B.Cu")
+		(net 6)
+	)
+	(segment
+		(start 170.2 93.7)
+		(end 171.5 93.7)
+		(width 1)
+		(layer "B.Cu")
+		(net 6)
+	)
+	(segment
 		(start 165 89.9925)
-		(end 167.7925 89.9925)
-		(width 1)
-		(layer "B.Cu")
-		(net 6)
-	)
-	(segment
-		(start 167.7925 89.9925)
-		(end 171.5 93.7)
+		(end 166.4925 89.9925)
 		(width 1)
 		(layer "B.Cu")
@@
 	)
 	(segment
-		(start 174 105)
-		(end 174 92.9)
+		(start 168.8 89.4)
+		(end 164.4 85)
+		(width 0.4)
+		(layer "F.Cu")
+		(net 9)
+	)
+	(segment
+		(start 164.4 85)
+		(end 162 85)
 		(width 0.4)
 		(layer "F.Cu")
@@
 	)
 	(segment
+		(start 170.1 89.4)
+		(end 168.8 89.4)
+		(width 0.4)
+		(layer "F.Cu")
+		(net 9)
+	)
+	(segment
+		(start 174 93.3)
+		(end 170.1 89.4)
+		(width 0.4)
+		(layer "F.Cu")
+		(net 9)
+	)
+	(segment
 		(start 158.6375 97.2625)
 		(end 157.175 97.2625)
@@
 	)
 	(segment
-		(start 166.1 85)
-		(end 162 85)
-		(width 0.4)
-		(layer "F.Cu")
-		(net 9)
-	)
-	(segment
 		(start 160.6 95.3)
 		(end 158.6375 97.2625)
@@
 	)
 	(segment
-		(start 174 92.9)
-		(end 166.1 85)
+		(start 174 105)
+		(end 174 93.3)
 		(width 0.4)
 		(layer "F.Cu")
 		(net 9)
+	)
+	(segment
+		(start 175.5 105.5)
+		(end 175.5 93.5)
+		(width 0.4)
+		(layer "F.Cu")
+		(net 10)
 	)
 	(segment
@@
 	)
 	(segment
-		(start 160 83)
-		(end 158 85)
+		(start 158.7 83)
+		(end 158 83.7)
 		(width 0.4)
 		(layer "F.Cu")
@@
 	)
 	(segment
+		(start 175.5 93.5)
+		(end 170.2 88.2)
+		(width 0.4)
+		(layer "F.Cu")
+		(net 10)
+	)
+	(segment
 		(start 151 104)
 		(end 152 103)
@@
 	)
 	(segment
-		(start 165.7 83)
-		(end 160 83)
-		(width 0.4)
-		(layer "F.Cu")
-		(net 10)
-	)
-	(segment
-		(start 175.5 92.8)
-		(end 165.7 83)
+		(start 158 83.7)
+		(end 158 85)
+		(width 0.4)
+		(layer "F.Cu")
+		(net 10)
+	)
+	(segment
+		(start 164.1 83)
+		(end 158.7 83)
 		(width 0.4)
 		(layer "F.Cu")
@@
 	)
 	(segment
-		(start 175.5 105.5)
-		(end 175.5 92.8)
+		(start 169.3 88.2)
+		(end 164.1 83)
+		(width 0.4)
+		(layer "F.Cu")
+		(net 10)
+	)
+	(segment
+		(start 170.2 88.2)
+		(end 169.3 88.2)
 		(width 0.4)
 		(layer "F.Cu")
@@
 	)
 	(segment
-		(start 166.5925 92.9925)
-		(end 167.0925 93.4925)
+		(start 161.1 101.6)
+		(end 166.5 96.2)
 		(width 0.4)
 		(layer "F.Cu")
@@
 	)
 	(segment
-		(start 165 92.9925)
-		(end 166.5925 92.9925)
+		(start 169 94.9)
+		(end 169 93.4925)
 		(width 0.4)
 		(layer "F.Cu")
@@
 	)
 	(segment
-		(start 167.0925 93.4925)
-		(end 169 93.4925)
-		(width 0.4)
-		(layer "F.Cu")
+		(start 159.6 101.6)
+		(end 161.1 101.6)
+		(width 0.4)
+		(layer "F.Cu")
+		(net 11)
+	)
+	(segment
+		(start 167.7 96.2)
+		(end 169 94.9)
+		(width 0.4)
+		(layer "F.Cu")
+		(net 11)
+	)
+	(segment
+		(start 166.5 96.2)
+		(end 167.7 96.2)
+		(width 0.4)
+		(layer "F.Cu")
