File: 0002-clap-detector/0002-clap-detector.kicad_pcb (KiCad board)
At the start: 2 copper layers, 58 x 37 mm, 49 parts, among them J1 9V, J2 OUT, K1 HF49FD 012-1H11, Q1 BC847B, Q2 BC847B, Q3 BCV26, Q4 BC847B, U1 4017

Commit message: Cleanup
Parts:
- removed the REF** at (164.0, 114.0)
- removed the REF** at (164.0, 112.0)
- added REF**: TestPoint_THTPad_D1.5mm_Drill0.7mm, TestPoint:TestPoint_THTPad_D1.5mm_Drill0.7mm, F.Cu at (129.9, 114.1)
- moved REF** 0.70 mm to (123.0, 90.3)
- moved REF** 0.20 mm to (175.4, 89.6)
- moved D2 0.10 mm to (173.0, 107.1)
Routing:
- net Net-(Q1-B): track 41.7 -> 40.5 mm
- net Net-(D2-A): track 76.7 -> 77.2 mm

Commit message: PCB - small correction
Routing:
- net Net-(MK1-+): track 39.3 -> 46.1 mm
Changed lines of the file:
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@@
 	)
 	(segment
-		(start 139.5 97.5)
-		(end 134.6 97.5)
+		(start 131.1 95)
+		(end 131.5 95.4)
 		(width 0.4)
 		(layer "F.Cu")
@@
 	)
 	(segment
-		(start 145 92)
-		(end 139.5 97.5)
+		(start 144.3 99.2)
+		(end 144.3 93.9)
 		(width 0.4)
 		(layer "F.Cu")
@@
 	)
 	(segment
-		(start 132.1 95)
-		(end 130 95)
+		(start 130 95)
+		(end 131.1 95)
+		(width 0.4)
+		(layer "F.Cu")
+		(net 2)
+	)
+	(segment
+		(start 131.5 99.2)
+		(end 132.1 99.8)
+		(width 0.4)
+		(layer "F.Cu")
+		(net 2)
+	)
+	(segment
+		(start 144.3 93.9)
+		(end 145 93.2)
 		(width 0.4)
 		(layer "F.Cu")
@@
 		(end 130 95)
 		(width 0.5)
+		(layer "F.Cu")
+		(net 2)
+	)
+	(segment
+		(start 131.5 95.4)
+		(end 131.5 99.2)
+		(width 0.4)
 		(layer "F.Cu")
 		(net 2)
@@
 	)
 	(segment
-		(start 134.6 97.5)
-		(end 132.1 95)
+		(start 132.1 99.8)
+		(end 143.7 99.8)
+		(width 0.4)
+		(layer "F.Cu")
+		(net 2)
+	)
+	(segment
+		(start 145 93.2)
+		(end 145 92)
+		(width 0.4)
+		(layer "F.Cu")
+		(net 2)
+	)
+	(segment
+		(start 143.7 99.8)
+		(end 144.3 99.2)
 		(width 0.4)
 		(layer "F.Cu")
@@
 	)
 	(segment
-		(start 144.36 94.54)
-		(end 138 94.54)
+		(start 142.8 92)
+		(end 140.26 94.54)
 		(width 0.4)
 		(layer "B.Cu")
@@
 	(segment
 		(start 145 92)
-		(end 145 93.9)
+		(end 142.8 92)
 		(width 0.4)
 		(layer "B.Cu")
@@
 	)
 	(segment
-		(start 145 93.9)
-		(end 144.36 94.54)
+		(start 140.26 94.54)
+		(end 138 94.54)
 		(width 0.4)
 		(layer "B.Cu")
